Commit message: Setting up own repository for the assignment in order to track changes and progress for assignment

File: roomba_one/lab_one/src/description/camera.xacro (robot description, xacro)
@@ -25,4 +25,5 @@
         <child link="camera_link_optical"/>
         <origin xyz="0 0 0" rpy="${-pi/2} 0 ${-pi/2}"/>
+        <origin xyz="0 0 0" rpy="${-pi/2} ${pi/9} ${-pi/2}"/>
     </joint>
     <link name="camera_link_optical"></link>
@@ -34,5 +35,5 @@
             <update_rate>10</update_rate>
             <camera>
-                <horizontal_fov>1.57</horizontal_fov> <!--90 degree fov-->
+                <horizontal_fov>2.0944</horizontal_fov> <!--90 degree fov-->
                 <image>
                     <format>R8G8B8</format>
@@ -42,9 +43,9 @@
                 <clip>
                     <near>0.05</near>
-                    <far>8.0</far>
+                    <far>20.0</far>
                 </clip>
                 <distortion>
-                  <k1>-0.1</k1> <!-- Radial distortion coefficient -->
-                  <k2>0.12</k2>  <!-- Radial distortion coefficient -->
+                  <k1>0.2</k1> <!-- Radial distortion coefficient -->
+                  <k2>0.0</k2>  <!-- Radial distortion coefficient -->
                   <k3>0.0</k3>   <!-- Sometimes used for higher-order distortion -->
                   <p1>0.0</p1>   <!-- Tangential distortion coefficient -->
@@ -52,4 +53,9 @@
                   <center>0.5 0.5</center> <!-- Distortion center in normalized coordinates -->
                 </distortion>
+                <noise>
+                    <type>gaussian</type>
+                    <mean>0.0</mean>
+                    <stddev>0.01</stddev>
+                </noise>
             </camera>
             <plugin name="camera_controller" filename="libgazebo_ros_camera.so">

File: roomba_one/lab_one/src/description/lidar.xacro (robot description, xacro)
@@ -34,9 +34,9 @@
             <pose> 0 0 0 0 0 0 </pose>
             <visualize>true</visualize>
-            <update_rate>10</update_rate>
+            <update_rate>5</update_rate>
             <ray>
                 <scan>
                     <horizontal>
-                        <samples>60</samples>
+                        <samples>180</samples>
                         <min_angle>-3.14</min_angle>
                         <max_angle>3.14</max_angle>
@@ -44,7 +44,12 @@
                 </scan>
                 <range>
-                    <min>0.3</min>
-                    <max>12</max>
+                    <min>0.1</min>
+                    <max>15</max>
                 </range>
+                <noise>
+                    <type>gaussian</type>
+                    <mean>0.0</mean>
+                    <stddev>0.03</stddev>
+                </noise>
             </ray>
             <plugin name="laser_controller" filename="libgazebo_ros_ray_sensor.so">

File: roomba_one/lab_one/src/description/robot.urdf.xacro (robot description, xacro)
@@ -1,5 +1,15 @@
 <?xml version="1.0"?>
 <robot xmlns:xacro="http://www.ros.org/wiki/xacro"  name="robot">
+    <xacro:arg name="use_ros2_control" default="true"/>
     <xacro:arg name="sim_mode" default="false"/>
     <xacro:include filename="robot_core.xacro" />
+    <xacro:if value="$(arg use_ros2_control)">
+        <xacro:include filename="ros2_control.xacro" />
+    </xacro:if>
+    <xacro:unless value="$(arg use_ros2_control)">
+        <xacro:include filename="gazebo_control.xacro" />
+    </xacro:unless>
+    <xacro:include filename="lidar.xacro" />
+    <xacro:include filename="camera.xacro" />
+    <xacro:include filename="depth_camera.xacro" />
 </robot>

File: roomba_one/lab_one/src/description/robot_core.xacro (robot description, xacro)
@@ -2,9 +2,29 @@
 <robot xmlns:xacro="http://www.ros.org/wiki/xacro" >
     <xacro:include filename="inertial_macros.xacro"/>
+    <xacro:property name="chassis_length" value="0.15"/>
+    <xacro:property name="chassis_width" value="0.1"/>
+    <xacro:property name="chassis_height" value="0.25"/>
+    <xacro:property name="chassis_mass" value="1.0"/>
+    <xacro:property name="wheel_radius" value="0.055"/>
+    <xacro:property name="wheel_thickness" value="0.026"/>
+    <xacro:property name="wheel_mass" value="0.05"/>
+    <xacro:property name="wheel_offset_x" value="-0.1"/>
+    <xacro:property name="wheel_offset_y" value="0.020"/>
+    <xacro:property name="wheel_offset_z" value="0.005"/>
+    <xacro:property name="caster_wheel_radius" value="0.048"/>
+    <xacro:property name="caster_wheel_mass" value="0.01"/>
+    <xacro:property name="caster_wheel_offset_x" value="0.05"/>
+    <xacro:property name="caster_wheel_offset_z" value="${wheel_offset_z - wheel_radius + caster_wheel_radius}"/>
     <!-- Define Roomba-style robot properties. Example below shows the structure used to define xacro properties -->
-    <xacro:property name="chassis_radius" value="0.18"/> <!-- Define all other required parameters in the same format -->
+    <xacro:property name="chassis_radius" value="0.127"/> <!-- Define all other required parameters in the same format -->
 	<!-- Define material colours. An example for white is shown below -->
     <material name="white">
         <color rgba="1 1 1 1" />
+    </material>
+    <material name="blue">
+        <color rgba="0 0 1 1" />
+    </material>
+    <material name="red">
+        <color rgba="1 0 0 1" />
     </material>
 	<!-- Define all of the robot links (base_link, chassis_link, wheels) -->
@@ -30,7 +50,7 @@
             <origin xyz="0 0 0.05"/>
             <geometry>
-                <cylinder radius="0.5" length="0.1"/>
+                <cylinder radius="0.3" length="0.1"/>
             </geometry>
-            <material name="white"/>
+            <material name="red"/>
         </visual>
         <collision>
@@ -48,5 +68,81 @@
     </gazebo>
     <!-- LEFT WHEEL LINK -->
+      <joint name="left_wheel_joint" type="continuous">
+        <parent link="base_link"/>
+        <child link="left_wheel"/>
+        <origin xyz="${wheel_offset_x} ${wheel_offset_y} 0" rpy="-${pi/2} 0 0" />
+        <axis xyz="0 0 1"/>
+    </joint>
+    <link name="left_wheel">
+        <visual>
+            <geometry>
+                <cylinder radius="${wheel_radius}" length="${wheel_thickness}"/>
+            </geometry>
+            <material name="blue"/>
+        </visual>
+        <collision>
+            <geometry>
+                <sphere radius="${wheel_radius}"/>
+            </geometry>
+        </collision>
+        <xacro:inertial_cylinder mass="${wheel_mass}" length="${wheel_thickness}" radius="${wheel_radius}">
+            <origin xyz="0 0 0" rpy="0 0 0"/>
+        </xacro:inertial_cylinder>
+    </link>
+    <gazebo reference="left_wheel">
+        <material>Gazebo/Blue</material>
+    </gazebo>
     <!-- RIGHT WHEEL LINK -->
+     <joint name="right_wheel_joint" type="continuous">
+        <parent link="base_link"/>
+        <child link="right_wheel"/>
+        <origin xyz="${wheel_offset_x} ${-wheel_offset_y} 0" rpy="${pi/2} 0 0" />
+        <axis xyz="0 0 -1"/>
+    </joint>
+    <link name="right_wheel">
+        <visual>
+            <geometry>
+                <cylinder radius="${wheel_radius}" length="${wheel_thickness}"/>
+            </geometry>
+            <material name="blue"/>
+        </visual>
+        <collision>
+            <geometry>
+                <sphere radius="${wheel_radius}"/>
+            </geometry>
+        </collision>
+        <xacro:inertial_cylinder mass="${wheel_mass}" length="${wheel_thickness}" radius="${wheel_radius}">
+            <origin xyz="0 0 0" rpy="0 0 0"/>
+        </xacro:inertial_cylinder>
+    </link>
+    <gazebo reference="right_wheel">
+        <material>Gazebo/Blue</material>
+    </gazebo>
     <!-- CASTER WHEEL LINK -->
+    <joint name="caster_wheel_joint" type="fixed">
+        <parent link="chassis"/>
+        <child link="caster_wheel"/>
+        <origin xyz="${caster_wheel_offset_x} 0 -.01"/>
+    </joint>
+    <link name="caster_wheel">
+        <visual>
+            <geometry>
+                <sphere radius="${caster_wheel_radius}"/>
+            </geometry>
+            <material name="white"/>
+        </visual>
+        <collision>
+            <geometry>
+                <sphere radius="${caster_wheel_radius}"/>
+            </geometry>
+        </collision>
+        <xacro:inertial_sphere mass="${caster_wheel_mass}" radius="${caster_wheel_radius}">
+            <origin xyz="0 0 0" rpy="0 0 0"/>
+        </xacro:inertial_sphere>
+    </link>
+    <gazebo reference="caster_wheel">
+        <material>Gazebo/White</material>
+        <mu1 value="0.001"/>
+        <mu2 value="0.001"/>
+    </gazebo>
 </robot>
