Commit message: Added start up file, adjusted robot to fit in doors, buid world and saved in lab_one woelds, changed Dockerfile

File: roomba_one/lab_one/src/description/robot_core.xacro (robot description, xacro)
@@ -2,5 +2,5 @@
 <robot xmlns:xacro="http://www.ros.org/wiki/xacro" >
     <xacro:include filename="inertial_macros.xacro"/>
-    <xacro:property name="chassis_length" value="0.15"/>
+    <xacro:property name="chassis_length" value="0.1"/>
     <xacro:property name="chassis_width" value="0.1"/>
     <xacro:property name="chassis_height" value="0.25"/>
@@ -10,9 +10,9 @@
     <xacro:property name="wheel_mass" value="0.05"/>
     <xacro:property name="wheel_offset_x" value="-0.1"/>
-    <xacro:property name="wheel_offset_y" value="0.020"/>
+    <xacro:property name="wheel_offset_y" value="0.17"/>
     <xacro:property name="wheel_offset_z" value="0.005"/>
     <xacro:property name="caster_wheel_radius" value="0.048"/>
     <xacro:property name="caster_wheel_mass" value="0.01"/>
-    <xacro:property name="caster_wheel_offset_x" value="0.05"/>
+    <xacro:property name="caster_wheel_offset_x" value="0.1"/>
     <xacro:property name="caster_wheel_offset_z" value="${wheel_offset_z - wheel_radius + caster_wheel_radius}"/>
     <!-- Define Roomba-style robot properties. Example below shows the structure used to define xacro properties -->
@@ -50,5 +50,5 @@
             <origin xyz="0 0 0.05"/>
             <geometry>
-                <cylinder radius="0.3" length="0.1"/>
+                <cylinder radius="0.2" length="0.1"/>
             </geometry>
             <material name="red"/>
@@ -57,5 +57,5 @@
             <origin xyz="0 0 0.05"/>
             <geometry>
-                <cylinder radius="0.5" length="0.1"/>
+                <cylinder radius="0.2" length="0.1"/>
             </geometry>
         </collision>
