Commit message: Created new mao and serialised it and made a few adjustments to the yaml for caster wheel and lidar for efficiency

File: roomba_one/lab_one/src/description/lidar.xacro (robot description, xacro)
@@ -33,10 +33,10 @@
         <sensor name="laser" type="ray">
             <pose> 0 0 0 0 0 0 </pose>
-            <visualize>true</visualize>
-            <update_rate>5</update_rate>
+            <visualize>false</visualize>
+            <update_rate>15</update_rate>
             <ray>
                 <scan>
                     <horizontal>
-                        <samples>180</samples>
+                        <samples>181</samples>
                         <min_angle>-3.14</min_angle>
                         <max_angle>3.14</max_angle>
@@ -44,12 +44,7 @@
                 </scan>
                 <range>
-                    <min>0.1</min>
-                    <max>15</max>
+                    <min>0.3</min>
+                    <max>6</max>
                 </range>
-                <noise>
-                    <type>gaussian</type>
-                    <mean>0.0</mean>
-                    <stddev>0.03</stddev>
-                </noise>
             </ray>
             <plugin name="laser_controller" filename="libgazebo_ros_ray_sensor.so">

File: roomba_one/lab_one/src/description/robot_core.xacro (robot description, xacro)
@@ -123,5 +123,5 @@
         <parent link="chassis"/>
         <child link="caster_wheel"/>
-        <origin xyz="${caster_wheel_offset_x} 0 -.01"/>
+        <origin xyz="${caster_wheel_offset_x} 0 ${caster_wheel_offset_z}"/>
     </joint>
     <link name="caster_wheel">
